File: Hardware/SMT/LFOVoltGenerator_SMT.sch (KiCad schematic (older format))
At the start: 46 parts

Commit message: correction
Parts:
- removed U_DIGPOT1: MCP41050, symbol MCP41050
- added C_BP2, C_BP4: 100nF, Capacitors_SMD:C_0805_HandSoldering, symbol C
- added C_BP3: 1uF, Capacitors_SMD:C_0805_HandSoldering, symbol C
- added R_OA_FB1: 10K, Resistors_SMD:R_0805_HandSoldering, symbol R
- added R_OA_GAIN1: 5K6, Resistors_SMD:R_0805_HandSoldering, symbol R
- added R_OA_GAIN2: 12K, Resistors_SMD:R_0805_HandSoldering, symbol R
- added SW_OAGAIN1: SW_SPDT, C&K_8_6mm_SPDT_ONON:C&K_8_6mm_SPDT_ONON, symbol SW_SPDT
- added U_OUT_DAC1: MCP4921, Housings_SOIC:SOIC-8_3.9x4.9mm_Pitch1.27mm, symbol MCP4921
- added U_OUT_OA1: MCP601-xSN, Housings_SOIC:SOIC-8_3.9x4.9mm_Pitch1.27mm, symbol MCP601-xSN
- R_FUNC1: value 1K -> 10K
Connections:
- net RING_SIGOUT is gone; now on net +5V: J_OUT1.2
- net SLEEVE_SIGOUT is gone; now on net GND: J_OUT1.3
- net +5V: now also C_BP2.1, C_BP3.1, C_BP4.1, U_OUT_DAC1.1 (Vdd), U_OUT_DAC1.6 (Vref), U_OUT_OA1.7 (V+)
- net DACCS: now also U_OUT_DAC1.2 (~CS)
- net GND: now also C_BP2.2, C_BP3.2, C_BP4.2, R_OA_GAIN1.1, R_OA_GAIN2.1, U_OUT_DAC1.5 (~LDAC), U_OUT_DAC1.7 (Vss), U_OUT_OA1.4 (V-)
- net MOSI: now also U_OUT_DAC1.4 (SDI)
- net SCK: now also U_OUT_DAC1.3 (SCK)
- net SW_FUNC: now also U_AVR1.30 ((PCINT16/RXD)PD0); no longer U_AVR1.9 ((PCINT21/OC0B/T1)PD5)
- net OA_SWEN: now reaches SW_EN1.5 (B)
- net OA_SWEN: now also R_OA_FB1.1, U_OUT_OA1.6
- net TIP_SIGOUT renamed SWEN_OUT
- new net: R_OA_FB1.2, SW_OAGAIN1.2 (B), U_OUT_OA1.2 (-)
- new net: R_OA_GAIN1.2, SW_OAGAIN1.1 (A)
- new net: R_OA_GAIN2.2, SW_OAGAIN1.3 (C)
- new net DAC_OA: U_OUT_DAC1.8 (Vout), U_OUT_OA1.3 (+)
Other:
- note added: "Selects either 5V(default) or 3V3 output"
- note removed: "ONLY USED FOR ISP"
- moved on the sheet: C_AVRCLK1, C_AVRCLK2, C_BP5, C_DB1, J_AUX2MAIN1, J_ISP1, J_MAIN2AUX1, J_OUT1, R_DB1, R_FREQ1, R_FUNC1, R_MUXIN1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
